Commit message: added gazebo differential drive plugin and correct joint axes direction

File: wheelchair_description/urdf/wheelchair.urdf (robot description, URDF)
Before this commit: robot wheelchair, 8 links, 7 joints
Links:
- removed link dummy
Joints:
- removed joint dummy_joint
- joint SwingL_rev: axis 0 -1 0 -> 0 1 0
- joint WheelR_cont: axis 0 -1 0 -> 0 1 0

Commit message: corected swing L and R inertial data

File: wheelchair_description/urdf/wheelchair.urdf (robot description, URDF)
Before this commit: robot wheelchair, 7 links, 6 joints
Links:
- link SwingL: mass 3.4241 -> 4.8363
Joints:
- joint SwingL_rev: limit lower=0 upper=0.67265 effort=0 velocity=2 -> lower=-0.51732 upper=0.15533 effort=0 velocity=2
- joint SwingR_rev: limit lower=0 upper=0.67265 effort=0 velocity=2 -> lower=-0.51732 upper=0.15533 effort=0 velocity=2
- joint WheelF_cont: origin xyz=-0.0518843000619276 -0.00660668610975347 -0.1478026 rpy=0 0 0.126653383400985 -> xyz=-0.0518843000619276 -0.00660668610975347 -0.1478026 rpy=0 0 0.0

File: wheelchair_description/urdf/wheelchair.urdf.xacro (robot description, xacro)
@@ -7,5 +7,4 @@
   <xacro:include filename="$(find wheelchair_description)/urdf/wheelchair.gazebo.xacro" />
   <!--extra dummy link -->
-  <link name="Dummy" />
   <link name="Frame">
     <inertial>
@@ -47,8 +46,4 @@
     </collision>
   </link>
-  <joint name="dummy_joint" type="fixed">
-     <parent link="Dummy"/>
-     <child link="Frame"/>
-  </joint>
   <link name="Caster">
     <inertial>
@@ -269,15 +264,15 @@
     <inertial>
       <origin
-        xyz="-0.15869 -0.056844 -0.023612"
-        rpy="0 0 0" />
-      <mass
-        value="3.4241" />
-      <inertia
-        ixx="0.0064026"
-        ixy="0.00029746"
-        ixz="-0.002243"
-        iyy="0.012384"
-        iyz="1.5901E-05"
-        izz="0.0099363" />
+        xyz="-0.14883 -0.054597 -0.033745"
+        rpy="0 0 0" />
+      <mass
+        value="4.8363" />
+      <inertia
+        ixx="0.0094524"
+        ixy="0.00067415"
+        ixz="-0.0056619"
+        iyy="0.022613"
+        iyz="-3.9175E-05"
+        izz="0.018459" />
     </inertial>
     <visual>
