Commit message: created xacro files and a new launch file: wheelchair_world.launch

File: wheelchair_description/urdf/wheelchair.urdf.xacro (robot description, xacro)
@@ -3,8 +3,10 @@
      Commit Version: 1.5.1-0-g916b5db  Build Version: 1.5.7152.31018
      For more information, please see http://wiki.ros.org/sw_urdf_exporter -->
-<robot
-  name="wheelchair">
-  <link
-    name="Frame">
+<robot name="wheelchair" xmlns:xacro="http://ros.org/wiki/xacro">
+  <!-- Import all Gazebo-customization elements, including Gazebo colors -->
+  <xacro:include filename="$(find wheelchair_description)/urdf/wheelchair.gazebo.xacro" />
+  <!--extra dummy link -->
+  <link name="Dummy" />
+  <link name="Frame">
     <inertial>
       <origin
@@ -45,6 +47,9 @@
     </collision>
   </link>
-  <link
-    name="Caster">
+  <joint name="dummy_joint" type="fixed">
+     <parent link="Dummy"/>
+     <child link="Frame"/>
+  </joint>
+  <link name="Caster">
     <inertial>
       <origin
@@ -85,7 +90,5 @@
     </collision>
   </link>
-  <joint
-    name="Caster_cont"
-    type="continuous">
+  <joint name="Caster_cont" type="continuous">
     <origin
       xyz="0.5078 0 0.00635"
@@ -101,6 +104,5 @@
       velocity="20" />
   </joint>
-  <link
-    name="WheelF">
+  <link name="WheelF">
     <inertial>
       <origin
@@ -141,7 +143,5 @@
     </collision>
   </link>
-  <joint
-    name="WheelF_cont"
-    type="continuous">
+  <joint name="WheelF_cont"  type="continuous">
     <origin
       xyz="-0.0518843000619276 -0.00660668610975347 -0.1478026"
@@ -157,6 +157,5 @@
       velocity="20" />
   </joint>
-  <link
-    name="SwingR">
+  <link name="SwingR">
     <inertial>
       <origin
@@ -197,7 +196,5 @@
     </collision>
   </link>
-  <joint
-    name="SwingR_rev"
-    type="revolute">
+  <joint  name="SwingR_rev" type="revolute">
     <origin
       xyz="-0.106 -0.2118548 -0.0238887"
@@ -216,6 +213,5 @@
     <dynamics damping="0.7" friction="0.0"/>
   </joint>
-  <link
-    name="WheelR">
+  <link name="WheelR">
     <inertial>
       <origin
@@ -256,7 +252,5 @@
     </collision>
   </link>
-  <joint
-    name="WheelR_cont"
-    type="continuous">
+  <joint name="WheelR_cont" type="continuous">
     <origin
       xyz="-0.232195893808092 -0.0517862 -0.0361948462997351"
@@ -272,6 +266,5 @@
       velocity="16.25" />
   </joint>
-  <link
-    name="SwingL">
+  <link name="SwingL">
     <inertial>
       <origin
@@ -312,7 +305,5 @@
     </collision>
   </link>
-  <joint
-    name="SwingL_rev"
-    type="revolute">
+  <joint name="SwingL_rev" type="revolute">
     <origin
       xyz="-0.106 0.20947 -0.023889"
@@ -331,6 +322,5 @@
     <dynamics damping="0.7" friction="0.0"/>
   </joint>
-  <link
-    name="WheelL">
+  <link name="WheelL">
     <inertial>
       <origin
@@ -371,7 +361,5 @@
     </collision>
   </link>
-  <joint
-    name="WheelL_cont"
-    type="continuous">
+  <joint name="WheelL_cont" type="continuous">
     <origin
       xyz="-0.2322 0.054167 -0.036195"
@@ -387,40 +375,4 @@
       velocity="16.25" />
   </joint>
-  <gazebo>
-    <plugin name="differential_drive_controller"
-            filename="libgazebo_ros_diff_drive.so">
-      <leftJoint>WheelL_cont</leftJoint>
-      <rightJoint>WheelR_cont</rightJoint>
-      <!-- Robot frame to calculate odometry from, defaults to `base_footprint` -->
-      <wheelSeparation>0.52728</wheelSeparation>
-      <wheelDiameter>0.635</wheelDiameter>
-      <!-- Wheel acceleration, in rad/s^2, defaults to 0.0 rad/s^2 -->
-      <wheelAcceleration>1.0</wheelAcceleration>
-      <!-- Maximum torque which the wheels can produce, in Nm, defaults to 5 Nm -->
-      <wheelTorque>20</wheelTorque>
-      <!-- Topic to receive geometry_msgs/Twist message commands, defaults to `cmd_vel` -->
-      <commandTopic>cmd_vel</commandTopic>
-      <!-- Topic to publish nav_msgs/Odometry messages, defaults to `odom` -->
-      <odometryTopic>odom</odometryTopic>
-      <!-- Odometry frame, defaults to `odom` -->
-      <odometryFrame>odom</odometryFrame>
-      <!-- Robot frame to calculate odometry from, defaults to `base_footprint` -->
-      <robotBaseFrame>Frame</robotBaseFrame>
-      <!-- Odometry source, 0 for ENCODER, 1 for WORLD, defaults to WORLD -->
-      <odometrySource>1</odometrySource>
-      <!-- Set to true to publish transforms for the wheel links, defaults to false -->
-      <publishWheelTF>false                                                                                                                                                                                                                               </publishWheelTF>
-      <!-- Set to true to publish transforms for the odometry, defaults to true -->
-      <publishOdom>true</publishOdom>
-      <!-- Set to true to publish sensor_msgs/JointState on /joint_states for the wheel joints, defaults to false -->
-      <publishWheelJointState>true</publishWheelJointState>
-    </plugin>
-  </gazebo>
-  <gazebo>
-    <plugin name="joint_state_publisher"
-    filename="libgazebo_ros_joint_state_publisher.so">
-    <jointName>Caster_cont, WheelF_cont, SwingR_rev, SwingL_rev, WheelL_cont, WheelR_cont</jointName>
-    </plugin>
-  </gazebo>
   <transmission name="SwingL_trans">
     <type>transmission_interface/SimpleTransmission</type>
@@ -429,5 +381,5 @@
     </actuator>
     <joint name="SwingL_rev">
-      <hardwareInterface>EffortJointInterface</hardwareInterface>
+      <hardwareInterface>hardware_interface/EffortJointInterface</hardwareInterface>
     </joint>
   </transmission>
@@ -438,11 +390,6 @@
     </actuator>
     <joint name="SwingR_rev">
-      <hardwareInterface>EffortJointInterface</hardwareInterface>
+      <hardwareInterface>hardware_interface/EffortJointInterface</hardwareInterface>
     </joint>
   </transmission>
-  <gazebo>
-    <plugin name="gazebo_ros_control" filename="libgazebo_ros_control.so">
-      <robotNamespace>/wheelchair</robotNamespace>
-    </plugin>
-  </gazebo>
 </robot>

Commit message: added ramp to the model, cleaned up gazebo model, cleaned up urdf

File: wheelchair_description/urdf/wheelchair.urdf.xacro (robot description, xacro)
@@ -5,12 +5,7 @@
 <robot name="wheelchair" xmlns:xacro="http://ros.org/wiki/xacro">
   <!-- Import all Gazebo-customization elements, including Gazebo colors -->
-  <!-- <xacro:include filename="$(find wheelchair_description)/urdf/wheelchair.gazebo" /> -->
+  <xacro:include filename="$(find wheelchair_description)/urdf/wheelchair.gazebo" />
   <!--extra dummy link -->
-<!--   <link name="base_footprint"/>
-  <joint name="base_joint" type="fixed">
-    <parent link="base_footprint"/>
-    <child link="base_link"/>
-    <origin xyz="0.0 0.0 0.0" rpy="0 0 0"/>
-  </joint> -->
+  <link name="base_footprint"/>
   <link name="base_link">
     <inertial>
@@ -52,7 +47,4 @@
     </collision>
   </link>
-  <gazebo reference="base_link">
-    <turnGravityOff>false</turnGravityOff>
-  </gazebo>
   <link name="Caster">
     <inertial>
@@ -94,28 +86,4 @@
     </collision>
   </link>
-  <gazebo reference="Caster">
-    <material>Gazebo/Black</material>
-    <turnGravityOff>false</turnGravityOff>
-  </gazebo>
-  <joint name="Caster_cont" type="continuous">
-    <origin
-      xyz="0.5078 0 0.00635"
-      rpy="0 0 0" />
-    <parent
-      link="base_link" />
-    <child
-      link="Caster" />
-    <axis
-      xyz="0 0 1" />
-    <limit
-      effort="1000"
-      velocity="20" />
-  </joint>
-  <gazebo reference ="Caster_cont">
-    <mu1 value="200.0"/>
-    <mu2 value="100.0"/>
-    <kp value="10000000.0"/>
-    <kd value= "1.0"/>
-</gazebo>
   <link name="WheelF">
     <inertial>
@@ -157,27 +125,4 @@
     </collision>
   </link>
-  <gazebo reference="WheelF">
-    <turnGravityOff>false</turnGravityOff>
-  </gazebo>
-  <joint name="WheelF_cont"  type="continuous">
-    <origin
-      xyz="-0.0518843000619276 -0.00660668610975347 -0.1478026"
-      rpy="0 0 0.126653383400985" />
-    <parent
-      link="Caster" />
-    <child
-      link="WheelF" />
-    <axis
-      xyz="0 -1 0" />
-    <limit
-      effort="1000"
-      velocity="20" />
-  </joint>
-  <gazebo reference ="WheelF_cont">
-    <mu1 value="200.0"/>
-    <mu2 value="100.0"/>
-    <kp value="10000000.0"/>
-    <kd value= "1.0"/>
-  </gazebo>
   <link name="SwingR">
     <inertial>
@@ -219,30 +164,4 @@
     </collision>
   </link>
-  <gazebo reference="SwingR">
-    <turnGravityOff>false</turnGravityOff>
-  </gazebo>
-  <joint  name="SwingR_rev" type="revolute">
-    <origin
-      xyz="-0.106 -0.2118548 -0.0238887"
-      rpy="0 0 0" />
-    <parent
-      link="base_link" />
-    <child
-      link="SwingR" />
-    <axis
-      xyz="0 1 0" />
-    <limit
-      lower="-0.8"
-      upper="0.5"
-      effort="1000"
-      velocity="2" />
-    <dynamics damping="0.7" friction="0.0"/>
-  </joint>
-  <gazebo reference ="SwingR_rev">
-    <mu1 value="200.0"/>
-    <mu2 value="100.0"/>
-    <kp value="10000000.0"/>
-    <kd value= "1.0"/>
-  </gazebo>
   <link name="WheelR">
     <inertial>
@@ -284,27 +203,4 @@
     </collision>
   </link>
-  <gazebo reference="WheelR">
-    <turnGravityOff>false</turnGravityOff>
-  </gazebo>
-  <joint name="WheelR_cont" type="continuous">
-    <origin
-      xyz="-0.232195893808092 -0.0517862 -0.0361948462997351"
-      rpy="0 0 0" />
-    <parent
-      link="SwingR" />
-    <child
-      link="WheelR" />
-    <axis
-      xyz="0 1 0" />
-    <limit
-      effort="1000"
-      velocity="16.25" />
-  </joint>
-  <gazebo reference ="WheelR_cont">
-    <mu1 value="200.0"/>
-    <mu2 value="100.0"/>
-    <kp value="10000000.0"/>
-    <kd value= "1.0"/>
-  </gazebo>
   <link name="SwingL">
     <inertial>
@@ -346,30 +242,4 @@
     </collision>
   </link>
-  <gazebo reference="SwingL">
-    <turnGravityOff>false</turnGravityOff>
-  </gazebo>
-  <joint name="SwingL_rev" type="revolute">
-    <origin
-      xyz="-0.106 0.20947 -0.023889"
-      rpy="0 0 0" />
-    <parent
-      link="base_link" />
-    <child
-      link="SwingL" />
-    <axis
-      xyz="0 1 0" />
-    <limit
-      lower="-0.8"
-      upper="0.5"
-      effort="1000"
-      velocity="2" />
-    <dynamics damping="0.7" friction="0.0"/>
-  </joint>
-  <gazebo reference ="SwingL_rev">
-    <mu1 value="200.0"/>
-    <mu2 value="100.0"/>
-    <kp value="10000000.0"/>
-    <kd value= "1.0"/>
-  </gazebo>
   <link name="WheelL">
     <inertial>
@@ -411,7 +281,85 @@
     </collision>
   </link>
-  <gazebo reference="WheelL">
-    <turnGravityOff>false</turnGravityOff>
-  </gazebo>
+  <joint name="base_joint" type="fixed">
+    <parent link="base_footprint"/>
+    <child link="base_link"/>
+    <origin xyz="0.0 0.0 0.0" rpy="0 0 0"/>
+  </joint>
+  <joint name="Caster_cont" type="continuous">
+    <origin
+      xyz="0.5078 0 0.00635"
+      rpy="0 0 0" />
+    <parent
+      link="base_link" />
+    <child
+      link="Caster" />
+    <axis
+      xyz="0 0 1" />
+    <limit
+      effort="100"
+      velocity="10" />
+  </joint>
+  <joint name="WheelF_cont"  type="continuous">
+    <origin
+      xyz="-0.0518843000619276 -0.00660668610975347 -0.1478026"
+      rpy="0 0 0.126653383400985" />
+    <parent
+      link="Caster" />
+    <child
+      link="WheelF" />
+    <axis
+      xyz="0 -1 0" />
+    <limit
+      effort="100"
+      velocity="10" />
+  </joint>
+  <joint  name="SwingR_rev" type="revolute">
+    <origin
+      xyz="-0.106 -0.2118548 -0.0238887"
+      rpy="0 0 0" />
+    <parent
+      link="base_link" />
+    <child
+      link="SwingR" />
+    <axis
+      xyz="0 1 0" />
+    <limit
+      lower="-0.8"
+      upper="0.5"
+      effort="100"
+      velocity="2" />
+    <dynamics damping="1.0" friction="0.0"/>
+  </joint>
+  <joint name="WheelR_cont" type="continuous">
+    <origin
+      xyz="-0.232195893808092 -0.0517862 -0.0361948462997351"
+      rpy="0 0 0" />
+    <parent
+      link="SwingR" />
+    <child
+      link="WheelR" />
+    <axis
+      xyz="0 1 0" />
+    <limit
+      effort="100"
+      velocity="16.25" />
+  </joint>
+  <joint name="SwingL_rev" type="revolute">
+    <origin
+      xyz="-0.106 0.20947 -0.023889"
+      rpy="0 0 0" />
+    <parent
+      link="base_link" />
+    <child
+      link="SwingL" />
+    <axis
+      xyz="0 1 0" />
+    <limit
+      lower="-0.8"
+      upper="0.5"
+      effort="100"
+      velocity="2" />
+    <dynamics damping="1.0" friction="0.0"/>
+  </joint>
   <joint name="WheelL_cont" type="continuous">
     <origin
@@ -425,13 +373,7 @@
       xyz="0 1 0" />
     <limit
-      effort="1000"
+      effort="100"
       velocity="16.25" />
   </joint>
-  <gazebo reference ="WheelL_cont">
-    <mu1 value="200.0"/>
-    <mu2 value="100.0"/>
-    <kp value="10000000.0"/>
-    <kd value= "1.0"/>
-  </gazebo>
   <!-- add transmission to swing arm joints -->
   <transmission name="SwingL_transmission">
@@ -476,14 +418,3 @@
     </joint>
   </transmission>
-  <gazebo>
-    <plugin name="gazebo_ros_control" filename= "libgazebo_ros_control.so">
-     <robotNamespace>/</robotNamespace>
-    </plugin>
-  </gazebo>
-  <gazebo>
-    <plugin name="joint_state_publisher"
-    filename="libgazebo_ros_joint_state_publisher.so">
-    <jointName>Caster_cont, WheelF_cont</jointName>
-    </plugin>
-  </gazebo>
 </robot>
