Commit message: modified twist controller, added output as graphs

File: wheelchair_description/urdf/wheelchair_2.0.urdf.xacro (robot description, xacro)
@@ -14,5 +14,5 @@
         rpy="0 0 0" />
       <mass
-        value="65.655" />
+        value="15.655" />
       <inertia
         ixx="0.18789"
@@ -313,4 +313,5 @@
       effort="0"
       velocity="10" />
+    <dynamics damping="1.0" friction="0.2"/>
   </joint>
   <joint  name="SwingR_rev" type="revolute">
@@ -344,4 +345,5 @@
       effort="43"
       velocity="16.25" />
+    <dynamics damping="1.0" friction="0.2"/>
   </joint>
   <joint name="SwingL_rev" type="revolute">
@@ -375,4 +377,5 @@
       effort="43"
       velocity="16.25" />
+    <dynamics damping="1.0" friction="0.2"/>
   </joint>
   <!-- add transmission to swing arm joints -->

Commit message: updated twist controller, csv file for twist commands, recording wheelchair_state in rosbag

File: wheelchair_description/urdf/wheelchair_2.0.urdf.xacro (robot description, xacro)
@@ -299,4 +299,5 @@
       effort="0"
       velocity="10" />
+    <dynamics damping="1.0" friction="0.2"/>
   </joint>
   <joint name="WheelF_cont"  type="continuous">

Commit message: added wheel_torque_controller and recording ft_sensor data

File: wheelchair_description/urdf/wheelchair_2.0.urdf.xacro (robot description, xacro)
@@ -314,5 +314,5 @@
       effort="0"
       velocity="10" />
-    <dynamics damping="1.0" friction="0.2"/>
+    <dynamics damping="1.0" friction="0.1"/>
   </joint>
   <joint  name="SwingR_rev" type="revolute">
@@ -346,5 +346,5 @@
       effort="43"
       velocity="16.25" />
-    <dynamics damping="1.0" friction="0.2"/>
+    <dynamics damping="1.0" friction="0.0"/>
   </joint>
   <joint name="SwingL_rev" type="revolute">
@@ -378,5 +378,5 @@
       effort="43"
       velocity="16.25" />
-    <dynamics damping="1.0" friction="0.2"/>
+    <dynamics damping="1.0" friction="0.0"/>
   </joint>
   <!-- add transmission to swing arm joints -->
@@ -409,5 +409,6 @@
     </actuator>
     <joint name="WheelL_cont">
-      <hardwareInterface>hardware_interface/VelocityJointInterface</hardwareInterface>
+      <!--hardwareInterface>hardware_interface/VelocityJointInterface</hardwareInterface-->
+      <hardwareInterface>hardware_interface/EffortJointInterface</hardwareInterface>
     </joint>
   </transmission>
@@ -419,5 +420,6 @@
     </actuator>
     <joint name="WheelR_cont">
-      <hardwareInterface>hardware_interface/VelocityJointInterface</hardwareInterface>
+      <!--hardwareInterface>hardware_interface/VelocityJointInterface</hardwareInterface-->
+      <hardwareInterface>hardware_interface/EffortJointInterface</hardwareInterface>
     </joint>
   </transmission>

Commit message: updating all files

File: wheelchair_description/urdf/wheelchair_2.0.urdf.xacro (robot description, xacro)
@@ -343,6 +343,7 @@
     <axis
       xyz="0 1 0" />
-    <limit
-      effort="43"
+    <!-- effort actual value is 43 -->
+    <limit
+      effort="1000"
       velocity="16.25" />
     <dynamics damping="1.0" friction="0.0"/>
@@ -375,6 +376,7 @@
     <axis
       xyz="0 1 0" />
-    <limit
-      effort="43"
+    <!-- effort actual value is 43 -->
+    <limit
+      effort="1000"
       velocity="16.25" />
     <dynamics damping="1.0" friction="0.0"/>
@@ -409,6 +411,6 @@
     </actuator>
     <joint name="WheelL_cont">
-      <!-- <hardwareInterface>hardware_interface/VelocityJointInterface</hardwareInterface> -->
-      <hardwareInterface>hardware_interface/EffortJointInterface</hardwareInterface>
+      <hardwareInterface>hardware_interface/VelocityJointInterface</hardwareInterface>
+<!--       <hardwareInterface>hardware_interface/EffortJointInterface</hardwareInterface> -->
     </joint>
   </transmission>
@@ -420,6 +422,6 @@
     </actuator>
     <joint name="WheelR_cont">
-      <!-- <hardwareInterface>hardware_interface/VelocityJointInterface</hardwareInterface> -->
-      <hardwareInterface>hardware_interface/EffortJointInterface</hardwareInterface>
+      <hardwareInterface>hardware_interface/VelocityJointInterface</hardwareInterface>
+<!--       <hardwareInterface>hardware_interface/EffortJointInterface</hardwareInterface> -->
     </joint>
   </transmission>
