Commit message: updated friction coefs wheelchair0.0

File: wheelchair_description/urdf/wheelchair_0.0.urdf.xacro (robot description, xacro)
@@ -137,4 +137,36 @@
 	    <origin xyz="0.0 0.0 0.0" rpy="0 0 0"/>
   	</joint>
+	<joint name="Wheelchair-base-Left-Caster-Yaw" type="continuous">
+	   <parent link="base_link"/>
+	   <child link="Left-Caster-Yaw"/>
+	   <origin xyz="0.35956 0.24291 0.1517"/>
+	   <axis xyz="0 0 -1"/>
+	   <limit effort= "100" lower = "${lower}" upper = "${upper}" velocity = "10"/>
+	   <dynamics damping = "0.7" friction ="1.5"/>
+	</joint>
+	<joint name="Wheelchair-base-Right-Caster-Yaw" type="continuous">
+	   <parent link="base_link"/>
+	   <child link="Right-Caster-Yaw"/>
+	   <origin xyz="0.35956 -0.24291 0.1517"/>
+	   <axis xyz="0 0 1"/>
+	   <limit effort= "100" lower = "${lower}" upper = "${upper}" velocity = "10"/>
+	   <dynamics damping = "0.7" friction ="1.5"/>
+	</joint>
+	<joint name="WheelL_cont" type="continuous">
+	   <parent link="base_link"/>
+	   <child link="Left-Wheel"/>
+	   <origin xyz="-0 0.26808 0.305"/>
+	   <axis xyz="0 1 0"/>
+	   <limit effort= "100" lower = "${lower}" upper = "${upper}" velocity = "10"/>
+	   <dynamics damping = "1.0" friction ="0.00263"/>
+	</joint>
+	<joint name="WheelR_cont" type="continuous">
+	   <parent link="base_link"/>
+	   <child link="Right-Wheel"/>
+	   <origin xyz="0 -0.26808 0.305"/>
+	   <axis xyz="0 1 0"/>
+	   <limit effort= "100" lower = "${lower}" upper = "${upper}" velocity = "10"/>
+	   <dynamics damping = "1.0" friction ="0.00263"/>
+	</joint>
 	<joint name="Left-Caster-Yaw-Left-Caster-Wheel" type="continuous">
 	   <parent link="Left-Caster-Yaw"/>
@@ -143,21 +175,5 @@
 	   <axis xyz="0 1 0"/>
 	   <limit effort= "10" lower = "${lower}" upper = "${upper}" velocity = "10"/>
-	   <dynamics damping = ".7" friction ="1.5"/>
-	</joint>
-	<joint name="Wheelchair-base-Left-Caster-Yaw" type="continuous">
-	   <parent link="base_link"/>
-	   <child link="Left-Caster-Yaw"/>
-	   <origin xyz="0.35956 0.24291 0.1517"/>
-	   <axis xyz="0 0 -1"/>
-	   <limit effort= "100" lower = "${lower}" upper = "${upper}" velocity = "10"/>
-	   <dynamics damping = "0.7" friction ="1.5"/>
-	</joint>
-	<joint name="WheelL_cont" type="continuous">
-	   <parent link="base_link"/>
-	   <child link="Left-Wheel"/>
-	   <origin xyz="-0 0.26808 0.305"/>
-	   <axis xyz="0 1 0"/>
-	   <limit effort= "100" lower = "${lower}" upper = "${upper}" velocity = "10"/>
-	   <dynamics damping = "0.7" friction ="1.5"/>
+	   <dynamics damping = ".0" friction ="0.000918"/>
 	</joint>
 	<joint name="Right-Caster-Yaw-Right-Caster-Wheel" type="continuous">
@@ -167,20 +183,5 @@
 	   <axis xyz="0 1 0"/>
 	   <limit effort= "100" lower = "${lower}" upper = "${upper}" velocity = "10"/>
-	</joint>
-	<joint name="Wheelchair-base-Right-Caster-Yaw" type="continuous">
-	   <parent link="base_link"/>
-	   <child link="Right-Caster-Yaw"/>
-	   <origin xyz="0.35956 -0.24291 0.1517"/>
-	   <axis xyz="0 0 1"/>
-	   <limit effort= "100" lower = "${lower}" upper = "${upper}" velocity = "10"/>
-	   <dynamics damping = "0.7" friction ="1.5"/>
-	</joint>
-	<joint name="WheelR_cont" type="continuous">
-	   <parent link="base_link"/>
-	   <child link="Right-Wheel"/>
-	   <origin xyz="0 -0.26808 0.305"/>
-	   <axis xyz="0 1 0"/>
-	   <limit effort= "100" lower = "${lower}" upper = "${upper}" velocity = "10"/>
-	   <dynamics damping = "0.7" friction ="1.5"/>
+	   <dynamics damping = ".0" friction ="0.000918"/>
 	</joint>
     <transmission name="Wheelchair_base_Left_Wheel-trans">

Commit message: changed twist to wheel velocity controller

File: wheelchair_description/urdf/wheelchair_0.0.urdf.xacro (robot description, xacro)
@@ -21,5 +21,5 @@
 			<origin rpy= "0 -0 0" xyz = "0.13 0 0.5"/>
 	    	<mass value="63.4"/>
-	     	<inertia ixx="3.853724" ixy="7e-06" ixz="0.022948" iyy="3.218409" iyz="7e-06" izz="5.782313"/>
+	     	<inertia ixx="3.853724" ixy="7e-06" ixz="0.022948" iyy="3.218409" iyz="7e-06" izz="5.02"/>
  	    </inertial>
   	</link>
@@ -143,5 +143,5 @@
 	   <axis xyz="0 0 -1"/>
 	   <limit effort= "100" lower = "${lower}" upper = "${upper}" velocity = "10"/>
-	   <dynamics damping = "0.7" friction ="1.5"/>
+	   <dynamics damping = "1.0" friction ="1.0"/>
 	</joint>
 	<joint name="Wheelchair-base-Right-Caster-Yaw" type="continuous">
@@ -151,5 +151,5 @@
 	   <axis xyz="0 0 1"/>
 	   <limit effort= "100" lower = "${lower}" upper = "${upper}" velocity = "10"/>
-	   <dynamics damping = "0.7" friction ="1.5"/>
+	   <dynamics damping = "1.0" friction ="1.0"/>
 	</joint>
 	<joint name="WheelL_cont" type="continuous">

Commit message: tested effort controllers

File: wheelchair_description/urdf/wheelchair_0.0.urdf.xacro (robot description, xacro)
@@ -142,6 +142,6 @@
 	   <origin xyz="0.35956 0.24291 0.1517"/>
 	   <axis xyz="0 0 -1"/>
-	   <limit effort= "100" lower = "${lower}" upper = "${upper}" velocity = "10"/>
-	   <dynamics damping = "1.0" friction ="1.0"/>
+	   <limit effort= "1000" velocity = "10"/>
+	   <dynamics damping = "0.0" friction ="1.0"/>
 	</joint>
 	<joint name="Wheelchair-base-Right-Caster-Yaw" type="continuous">
@@ -150,6 +150,6 @@
 	   <origin xyz="0.35956 -0.24291 0.1517"/>
 	   <axis xyz="0 0 1"/>
-	   <limit effort= "100" lower = "${lower}" upper = "${upper}" velocity = "10"/>
-	   <dynamics damping = "1.0" friction ="1.0"/>
+	   <limit effort= "1000" velocity = "10"/>
+	   <dynamics damping = "0.0" friction ="1.0"/>
 	</joint>
 	<joint name="WheelL_cont" type="continuous">
@@ -158,6 +158,6 @@
 	   <origin xyz="-0 0.26808 0.305"/>
 	   <axis xyz="0 1 0"/>
-	   <limit effort= "100" lower = "${lower}" upper = "${upper}" velocity = "10"/>
-	   <dynamics damping = "1.0" friction ="0.00263"/>
+	   <limit effort= "1000" velocity = "10"/>
+	   <dynamics damping = "0.0" friction ="0.00263"/>
 	</joint>
 	<joint name="WheelR_cont" type="continuous">
@@ -166,13 +166,13 @@
 	   <origin xyz="0 -0.26808 0.305"/>
 	   <axis xyz="0 1 0"/>
-	   <limit effort= "100" lower = "${lower}" upper = "${upper}" velocity = "10"/>
-	   <dynamics damping = "1.0" friction ="0.00263"/>
+	   <limit effort= "1000"  velocity = "10"/>
+	   <dynamics damping = "0.0" friction ="0.00263"/>
 	</joint>
 	<joint name="Left-Caster-Yaw-Left-Caster-Wheel" type="continuous">
 	   <parent link="Left-Caster-Yaw"/>
 	   <child link="Left-Caster-Wheel"/>
-	   <origin xyz="-0.04295 -0.00183 -0.0917"/>
-	   <axis xyz="0 1 0"/>
-	   <limit effort= "10" lower = "${lower}" upper = "${upper}" velocity = "10"/>
+	   <origin xyz="-0.03295 -0.00183 -0.0917"/>
+	   <axis xyz="0 1 0"/>
+	   <limit effort= "1000" velocity = "10"/>
 	   <dynamics damping = ".0" friction ="0.000918"/>
 	</joint>
@@ -180,7 +180,7 @@
 	   <parent link="Right-Caster-Yaw"/>
 	   <child link="Right-Caster-Wheel"/>
-	   <origin xyz="-0.04295 0.00183 -0.0917"/>
-	   <axis xyz="0 1 0"/>
-	   <limit effort= "100" lower = "${lower}" upper = "${upper}" velocity = "10"/>
+	   <origin xyz="-0.03295 0.00183 -0.0917"/>
+	   <axis xyz="0 1 0"/>
+	   <limit effort= "1000" velocity = "10"/>
 	   <dynamics damping = ".0" friction ="0.000918"/>
 	</joint>
@@ -188,9 +188,10 @@
       	<type>transmission_interface/SimpleTransmission</type>
       	<actuator name="Wheelchair_base_Left_Wheel-motor">
+      		<hardwareInterface>hardware_interface/EffortJointInterface</hardwareInterface>
         	<mechanicalReduction>1</mechanicalReduction>
      	</actuator>
       	<joint name="WheelL_cont">
-        	<hardwareInterface>hardware_interface/VelocityJointInterface</hardwareInterface>
-        	<!-- <hardwareInterface>hardware_interface/EffortJointInterface</hardwareInterface> -->
+        	<!-- <hardwareInterface>hardware_interface/VelocityJointInterface</hardwareInterface> -->
+        	<hardwareInterface>hardware_interface/EffortJointInterface</hardwareInterface>
       	</joint>
     </transmission>
@@ -198,9 +199,10 @@
       	<type>transmission_interface/SimpleTransmission</type>
       	<actuator name="Wheelchair_base_Right_Wheel-motor">
+      		<hardwareInterface>hardware_interface/EffortJointInterface</hardwareInterface>
         	<mechanicalReduction>1</mechanicalReduction>
       	</actuator>
       	<joint name="WheelR_cont">
-        	<hardwareInterface>hardware_interface/VelocityJointInterface</hardwareInterface>
-        	<!-- <hardwareInterface>hardware_interface/EffortJointInterface</hardwareInterface> -->
+        	<!-- <hardwareInterface>hardware_interface/VelocityJointInterface</hardwareInterface> -->
+        	<hardwareInterface>hardware_interface/EffortJointInterface</hardwareInterface>
       	</joint>
     </transmission>

Commit message: implemented joint_effort service call

File: wheelchair_description/urdf/wheelchair_0.0.urdf.xacro (robot description, xacro)
@@ -116,5 +116,5 @@
   	<link name="Right-Wheel">
 	  	<visual>
-	  		<origin rpy  = "0 -0 0" xyz = "0 0.26808 -0.305"/>
+	  		<origin rpy  = "0.0 0.0 0.0" xyz = "0.0 0.26808 -0.305"/>
 	  		<geometry>
 		  		<mesh scale=" 1 1 1" filename = "package://wheelchair_description/meshes/Right-Wheel.STL"/>
@@ -122,5 +122,5 @@
 	  	</visual>
 	  	<collision>
-        	<origin rpy  = "0 -0 0" xyz = "0 0.26808 -0.305"/>
+        	<origin rpy  = "0.0 0.0 0.0" xyz = "0.0 0.26808 -0.305"/>
         	<geometry>
           		<mesh scale=" 1 1 1" filename = "package://wheelchair_description/meshes/Right-Wheel_col.STL"/>
@@ -156,5 +156,5 @@
 	   <parent link="base_link"/>
 	   <child link="Left-Wheel"/>
-	   <origin xyz="-0 0.26808 0.305"/>
+	   <origin xyz="0.0 0.26808 0.305"/>
 	   <axis xyz="0 1 0"/>
 	   <limit effort= "1000" velocity = "10"/>
