Commit message: effort bug fixed in urdf - all controllers working properly

File: wheelchair_description/urdf/Archive/wheelchair.urdf (robot description, URDF)
Before this commit: robot wheelchair, 7 links, 6 joints
Links:
- removed link base_link
- added link Frame, mass 25.5218455226117; collision mesh filename=package://wheelchair/meshes/Frame.STL; visual mesh filename=package://wheelchair/meshes/Frame.STL
- link Caster: geometry collision mesh filename=package://wheelchair/meshes/Caster.STL; visual mesh filename=package://wheelchair/meshes/Caster.STL
- link SwingL: geometry collision mesh filename=package://wheelchair/meshes/SwingL.STL; visual mesh filename=package://wheelchair/meshes/SwingL.STL
- link SwingR: geometry collision mesh filename=package://wheelchair/meshes/SwingR.STL; visual mesh filename=package://wheelchair/meshes/SwingR.STL
- link WheelF: geometry collision mesh filename=package://wheelchair/meshes/WheelF.STL; visual mesh filename=package://wheelchair/meshes/WheelF.STL
- link WheelL: geometry collision mesh filename=package://wheelchair/meshes/WheelL.STL; visual mesh filename=package://wheelchair/meshes/WheelL.STL
- link WheelR: geometry collision mesh filename=package://wheelchair/meshes/WheelR.STL; visual mesh filename=package://wheelchair/meshes/WheelR.STL
Joints:
- joint Caster_cont: limit effort=1000 velocity=20 -> effort=0 velocity=20; parent base_link -> Frame
- joint SwingL_rev: limit lower=-0.8 upper=0.5 effort=1000 velocity=2 -> lower=-0.51732 upper=0.15533 effort=0 velocity=2; parent base_link -> Frame
- joint SwingR_rev: limit lower=-0.8 upper=0.5 effort=1000 velocity=2 -> lower=-0.51732 upper=0.15533 effort=0 velocity=2; parent base_link -> Frame
- joint WheelF_cont: limit effort=1000 velocity=20 -> effort=0 velocity=20; origin xyz=-0.0518843000619276 -0.00660668610975347 -0.1478026 rpy=0 0 0.126653383400985 -> xyz=-0.0518843000619276 -0.00660668610975347 -0.1478026 rpy=0 0 0.0
- joint WheelL_cont: limit effort=1000 velocity=16.25 -> effort=0 velocity=16.25
- joint WheelR_cont: limit effort=1000 velocity=16.25 -> effort=0 velocity=16.25

File: wheelchair_description/urdf/wheelchair.urdf (robot description, URDF)
Before this commit: robot wheelchair, 7 links, 6 joints
Links:
- removed link Frame
- added link base_footprint
- added link base_link, mass 25.5218455226117; collision mesh filename=package://wheelchair_description/meshes/Frame.STL; visual mesh filename=package://wheelchair_description/meshes/Frame.STL
- link Caster: geometry collision mesh filename=package://wheelchair_description/meshes/Caster.STL; visual mesh filename=package://wheelchair_description/meshes/Caster.STL
- link SwingL: geometry collision mesh filename=package://wheelchair_description/meshes/SwingL.STL; visual mesh filename=package://wheelchair_description/meshes/SwingL.STL
- link SwingR: geometry collision mesh filename=package://wheelchair_description/meshes/SwingR.STL; visual mesh filename=package://wheelchair_description/meshes/SwingR.STL
- link WheelF: geometry collision mesh filename=package://wheelchair_description/meshes/WheelF.STL; visual mesh filename=package://wheelchair_description/meshes/WheelF.STL
- link WheelL: geometry collision mesh filename=package://wheelchair_description/meshes/WheelL.STL; visual mesh filename=package://wheelchair_description/meshes/WheelL.STL
- link WheelR: geometry collision mesh filename=package://wheelchair_description/meshes/WheelR.STL; visual mesh filename=package://wheelchair_description/meshes/WheelR.STL
Joints:
- added joint base_joint: type fixed, parent base_footprint, child base_link, origin xyz=0.0 0.0 0.0 rpy=0 0 0
- joint Caster_cont: parent Frame -> base_link
- joint SwingL_rev: limit lower=-0.51732 upper=0.15533 effort=0 velocity=2 -> lower=0 upper=0.67265 effort=0 velocity=2; parent Frame -> base_link
- joint SwingR_rev: limit lower=-0.51732 upper=0.15533 effort=0 velocity=2 -> lower=0 upper=0.67265 effort=0 velocity=2; parent Frame -> base_link
- joint WheelF_cont: origin xyz=-0.0518843000619276 -0.00660668610975347 -0.1478026 rpy=0 0 0.0 -> xyz=-0.0518843000619276 -0.00660668610975347 -0.1478026 rpy=0 0 0.126653383400985
